File: PCB/ESPOut/Płytka.sch (EAGLE design)
At the start: 70 parts, among them IC1 L293D, IC2 LM2576S/5V, K1 G5L, K2 G5L, K3 G5L, K4 G5L, K5 G5L, Q1 AOD2922, Q2 AOD2922, Q3 AOD2922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

Commit message: Add new PCBs
Parts:
- C2: device rcl:CPOL-EUE2.5-6 -> rcl:CPOL-EUE3.5-8
- D3: device diode:1N4004 -> diode:1N5908
- IC2: device v-reg-3:LM2576S -> v-reg-3:LM2576T
- Q1, Q2, Q3, Q6, Q7: device transistor-power:IRF3704S -> Clean-Kong:MOSFET_NIXTY8N65X2
Other:
- moved on the sheet: Q1, Q2, Q3, Q6, Q7

Commit message: Creating charts
Parts:
- C1, C6: value (none) -> 100u
- C2, C3, C4, C5, C7, C8: value (none) -> 10u
- R1, R2, R25, R26, R3, R4, R5: value (none) -> 10K
- R10: value (none) -> 330
- R11, R12, R30: value (none) -> 100
Other:
- note added: "ESP Outputs"

Commit message: Add new method of controling the supply
Parts:
- removed C6: 100u, rcl:C-EUC0805K
- removed C7: 10u, rcl:C-EUC0805K
- removed U2: LM3940IMP-3.3, LM3940IMP-3.3:LM3940IMP-3.3
- added C9: (no value), rcl:C-EUC0805K
- added OK1: 4N35, optocoupler:4N35
- added R35, R36, R6: (no value), rcl:R-EU_R0805
Connections:
- new net EN_5V: R35.2
- new net N$15: IC2.OFF, OK1.COL, R6.1
- new net N$26: OK1.A, R35.1
- new net N$29: C9.2, OK1.BAS, R36.2
- net +3V3: no longer C7.1, U2.OUT
- net +5V: no longer C6.1, U2.IN
- net GND: now also C9.1, OK1.C, OK1.EMI, R36.1; no longer C6.2, C7.2, IC2.OFF, U2.GND
- net VCC: now also R6.2
Other:
- moved on the sheet: C1
