File: PCB/ESPSensor/Płytka.brd (EAGLE design)
At the start: 97.8 x 73.3 mm, 50 parts, among them IC2 LM2576S/5V, J1 HUM1, J2 HUM2, J3 TEMP, J4 SUN, Q4 BSS138, Q5 BSS138, U1 ESP-WROOM-32, U2 LM3940IMP-3.3

Commit message: no message
Parts:
- added SV1, SV3, SV4, SV5: (no value), con-lstb:MA04-1
Connections:
- removed net P1ON: U1.31
- removed net P2ON: U1.30
- net +3V3: now also J3.1, J4.1
- net +5V: no longer J3.1, J4.1
Changed lines of the file:
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@@
 <attribute name="VALUE" x="238.84" y="78.715" size="1.27" layer="28" rot="MR90" align="top-left"/>
+</element>
+<element name="SV1" library="con-lstb" library_urn="urn:adsk.eagle:library:162" package="MA04-1" package3d_urn="urn:adsk.eagle:package:8337/1" value="" x="-63.5" y="-69.215" smashed="yes">
+<attribute name="MF" value="" x="-63.5" y="-69.215" size="1.778" layer="27" display="off"/>
+<attribute name="MPN" value="" x="-63.5" y="-69.215" size="1.778" layer="27" display="off"/>
+<attribute name="NAME" x="-68.58" y="-67.564" size="1.27" layer="25" ratio="10"/>
+<attribute name="OC_FARNELL" value="unknown" x="-63.5" y="-69.215" size="1.778" layer="27" display="off"/>
+<attribute name="OC_NEWARK" value="unknown" x="-63.5" y="-69.215" size="1.778" layer="27" display="off"/>
+<attribute name="POPULARITY" value="41" x="-63.5" y="-69.215" size="1.778" layer="27" display="off"/>
+<attribute name="VALUE" x="-62.865" y="-67.564" size="1.27" layer="27" ratio="10"/>
+</element>
+<element name="SV3" library="con-lstb" library_urn="urn:adsk.eagle:library:162" package="MA04-1" package3d_urn="urn:adsk.eagle:package:8337/1" value="" x="-63.5" y="-74.93" smashed="yes">
+<attribute name="MF" value="" x="-63.5" y="-74.93" size="1.778" layer="27" display="off"/>
+<attribute name="MPN" value="" x="-63.5" y="-74.93" size="1.778" layer="27" display="off"/>
+<attribute name="NAME" x="-68.58" y="-73.279" size="1.27" layer="25" ratio="10"/>
+<attribute name="OC_FARNELL" value="unknown" x="-63.5" y="-74.93" size="1.778" layer="27" display="off"/>
+<attribute name="OC_NEWARK" value="unknown" x="-63.5" y="-74.93" size="1.778" layer="27" display="off"/>
+<attribute name="POPULARITY" value="41" x="-63.5" y="-74.93" size="1.778" layer="27" display="off"/>
+<attribute name="VALUE" x="-62.865" y="-73.279" size="1.27" layer="27" ratio="10"/>
+</element>
+<element name="SV4" library="con-lstb" library_urn="urn:adsk.eagle:library:162" package="MA04-1" package3d_urn="urn:adsk.eagle:package:8337/1" value="" x="-63.5" y="-80.645" smashed="yes">
+<attribute name="MF" value="" x="-63.5" y="-80.645" size="1.778" layer="27" display="off"/>
+<attribute name="MPN" value="" x="-63.5" y="-80.645" size="1.778" layer="27" display="off"/>
+<attribute name="NAME" x="-68.58" y="-78.994" size="1.27" layer="25" ratio="10"/>
+<attribute name="OC_FARNELL" value="unknown" x="-63.5" y="-80.645" size="1.778" layer="27" display="off"/>
+<attribute name="OC_NEWARK" value="unknown" x="-63.5" y="-80.645" size="1.778" layer="27" display="off"/>
+<attribute name="POPULARITY" value="41" x="-63.5" y="-80.645" size="1.778" layer="27" display="off"/>
+<attribute name="VALUE" x="-62.865" y="-78.994" size="1.27" layer="27" ratio="10"/>
+</element>
+<element name="SV5" library="con-lstb" library_urn="urn:adsk.eagle:library:162" package="MA04-1" package3d_urn="urn:adsk.eagle:package:8337/1" value="" x="-63.5" y="-86.36" smashed="yes">
+<attribute name="MF" value="" x="-63.5" y="-86.36" size="1.778" layer="27" display="off"/>
+<attribute name="MPN" value="" x="-63.5" y="-86.36" size="1.778" layer="27" display="off"/>
+<attribute name="NAME" x="-68.58" y="-84.709" size="1.27" layer="25" ratio="10"/>
+<attribute name="OC_FARNELL" value="unknown" x="-63.5" y="-86.36" size="1.778" layer="27" display="off"/>
+<attribute name="OC_NEWARK" value="unknown" x="-63.5" y="-86.36" size="1.778" layer="27" display="off"/>
+<attribute name="POPULARITY" value="41" x="-63.5" y="-86.36" size="1.778" layer="27" display="off"/>
+<attribute name="VALUE" x="-62.865" y="-84.709" size="1.27" layer="27" ratio="10"/>
 </element>
 </elements>
@@
 <contactref element="J1" pad="1"/>
 <contactref element="J2" pad="1"/>
-<contactref element="J3" pad="1"/>
-<contactref element="J4" pad="1"/>
 <contactref element="U2" pad="1"/>
 <wire x1="83.82" y1="45.18" x2="69.85" y2="68.58" width="0" layer="19" extent="1-1"/>
 <wire x1="83.82" y1="36.29" x2="83.82" y2="45.18" width="0" layer="19" extent="1-1"/>
-<wire x1="83.82" y1="27.4" x2="83.82" y2="36.29" width="0" layer="19" extent="1-1"/>
-<wire x1="83.82" y1="18.51" x2="83.82" y2="27.4" width="0" layer="19" extent="1-1"/>
 <wire x1="37.97" y1="64.77" x2="69.85" y2="68.58" width="0" layer="19" extent="1-1"/>
 <wire x1="26.67" y1="53.34" x2="37.97" y2="64.77" width="0" layer="19" extent="1-1"/>
@@
 <contactref element="LED1" pad="A"/>
 <wire x1="-69.53" y1="77.47" x2="-45.94" y2="77.47" width="0" layer="19" extent="1-1"/>
-</signal>
-<signal name="P1ON">
-<contactref element="U1" pad="31"/>
-</signal>
-<signal name="P2ON">
-<contactref element="U1" pad="30"/>
 </signal>
 <signal name="+3V3">
@@
 <contactref element="SV2" pad="1"/>
 <contactref element="U2" pad="3"/>
+<contactref element="J4" pad="1"/>
+<contactref element="J3" pad="1"/>
+<wire x1="83.82" y1="18.51" x2="83.82" y2="27.4" width="0" layer="19" extent="1-1"/>
+<wire x1="46.63" y1="46.37" x2="83.82" y2="27.4" width="0" layer="19" extent="1-1"/>
+<wire x1="140.65" y1="-46.99" x2="83.82" y2="18.51" width="0" layer="19" extent="1-1"/>
 <wire x1="140.65" y1="-52.07" x2="140.65" y2="-46.99" width="0" layer="19" extent="1-1"/>
 <wire x1="140.97" y1="-63.5" x2="140.65" y2="-52.07" width="0" layer="19" extent="1-1"/>
-<wire x1="46.63" y1="46.37" x2="140.65" y2="-46.99" width="0" layer="19" extent="1-1"/>
-<wire x1="201.61" y1="85.09" x2="140.65" y2="-46.99" width="0" layer="19" extent="1-1"/>
+<wire x1="201.61" y1="85.09" x2="83.82" y2="27.4" width="0" layer="19" extent="1-1"/>
 <wire x1="209.23" y1="100.33" x2="201.61" y2="85.09" width="0" layer="19" extent="1-1"/>
 <wire x1="209.23" y1="106.68" x2="209.23" y2="100.33" width="0" layer="19" extent="1-1"/>

Commit message: Add new PCBs
Parts:
- removed DISP, SV3, SV4, SV5: (no value), con-lstb:MA04-1
- added C14, C15, C3, C4, C5: (no value), rcl:C0805K
- added I2C_3V3_1, I2C_3V3_2, I2C_5V_1, I2C_5V_2: (no value), con-lstb:MA04-1
- added J5: K3, PUTRocketLab_connectors:W_TYPE_2MM_2_N
- added J6: K2, PUTRocketLab_connectors:W_TYPE_2MM_2_N
- added J7: K1, PUTRocketLab_connectors:W_TYPE_2MM_2_N
- added J8: K5, PUTRocketLab_connectors:W_TYPE_2MM_2_N
- added J9: K4, PUTRocketLab_connectors:W_TYPE_2MM_2_N
- added Q1, Q2, Q3, Q6, Q7: BSS138, bss138_10:SOT23
- added R1, R2, R3, R4, R5: (no value), rcl:R0805
- added R11, R12, R13, R31, R32, R33, R6, R7, R8, R9: 10k, rcl:R0805
- C2: device rcl:E2,5-6 -> rcl:E3,5-8
- D3: device diode:DO41-10 -> diode:C4111-15
- IC2: device v-reg-3:TO263-5 -> v-reg-3:TO220-5
- SV1: device con-lstb:MA04-1 -> con-lsta:FE05-1
- moved Q5 228.4 mm to (12.1, 14.0), turned to 270 degrees
- moved R29 224.2 mm to (14.6, 12.7), turned to 270 degrees
- moved R28 223.4 mm to (9.53, 11.8), turned to 270 degrees
- moved R27 216.0 mm to (9.53, 15.9), turned to 90 degrees
- moved R16 215.9 mm to (26.0, 14.0), turned to 90 degrees
- moved Q4 207.4 mm to (28.6, 12.7), turned to 90 degrees
- moved R15 205.1 mm to (31.1, 15.0), turned to 90 degrees
- moved R14 201.4 mm to (31.1, 10.8), turned to 270 degrees
- moved C6 190.3 mm to (55.4, 61.6)
- moved U2 189.8 mm to (53.3, 66.7)
- moved C7 188.8 mm to (51.8, 61.6)
- moved D4 181.8 mm to (11.4, 52.1), turned to 270 degrees
- moved D5 179.0 mm to (12.1, 40.6), turned to 270 degrees
- moved D6 176.1 mm to (13.3, 30.5), turned to 270 degrees
- moved D7 174.9 mm to (13.3, 21.6), turned to 270 degrees
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Connections:
- removed net P1: U1.13
- removed net P2: U1.14
- new net K1: Q3.2, R12.1, U1.31
- new net K2: Q1.2, R7.1, U1.30
- new net K3: Q2.2, R9.1, U1.29
- new net K4: Q7.2, R33.1, U1.28
- new net K5: Q6.2, R31.1, U1.27
- new net N$1: C5.1, J5.1, Q2.3, R1.1
- new net N$10: SV1.5, U1.8
- new net N$11: Q1.1, R6.1
- new net N$12: SV1.4, U1.9
- new net N$13: Q2.1, R8.1
- new net N$14: SV1.3, U1.10
- new net N$16: Q3.1, R11.1
- new net N$17: SV1.2, U1.11
- new net N$2: C4.1, J6.1, Q1.3, R2.1
- new net N$20: Q6.1, R13.1
- new net N$22: SV1.1, U1.12
- new net N$24: Q7.1, R32.1
- new net N$5: C3.1, J7.1, Q3.3, R3.1
- new net N$6: C14.1, J9.1, Q7.3, R5.1
- new net N$7: C15.1, J8.1, Q6.3, R4.1
- net +3V3: now also I2C_3V3_1.1, I2C_3V3_2.1, R11.2, R12.2, R13.2, R31.2, R32.2, R33.2, R6.2, R7.2, R8.2, R9.2
- net +5V: now also I2C_5V_1.1, I2C_5V_2.1, R1.2, R2.2, R3.2, R4.2, R5.2; no longer DISP.1
- net A3: now also U1.7
- net GND: now also C14.2, C15.2, C3.2, C4.2, C5.2, I2C_3V3_1.4, I2C_3V3_2.4, I2C_5V_1.4, I2C_5V_2.4, J5.2, J6.2, J7.2, J8.2, J9.2; no longer DISP.4
- net SCL: now also I2C_5V_1.2, I2C_5V_2.2
- net SCL_LV: now also I2C_3V3_1.2, I2C_3V3_2.2; no longer DISP.2
- net SDA: now also I2C_5V_1.3, I2C_5V_2.3
- net SDA_LV: now also I2C_3V3_1.3, I2C_3V3_2.3; no longer DISP.3
Routing:
- net +3V3: track 0.00 -> 248.8 mm, vias 0 -> 1
- net +5V: track 0.00 -> 246.4 mm, vias 0 -> 4
- net SCL_LV: track 0.00 -> 92.9 mm, vias 0 -> 1
- net SDA_LV: track 0.00 -> 91.4 mm, vias 0 -> 1
- net GND: track 0.00 -> 77.2 mm, vias 0 -> 6
- net A3: track 0.00 -> 48.3 mm
- net EN: track 0.00 -> 46.0 mm
- net N$19: track 0.00 -> 42.1 mm
- net A2: track 0.00 -> 39.6 mm
- net A0: track 0.00 -> 39.1 mm
- net IO0: track 0.00 -> 37.3 mm, vias 0 -> 1
- net SCL: track 0.00 -> 35.6 mm
- net A1: track 0.00 -> 32.8 mm
- net K1: track 0.00 -> 26.0 mm, vias 0 -> 2
- net SDA: track 0.00 -> 25.3 mm
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- added copper zone on layer 1, net GND
- added copper zone on layer 16, net GND
Other:
- board size 97.8 x 73.3 mm -> 75 x 71.2 mm
- board text added: "A. KRUSZYNSKI"
- board text added: "C.KULCZYK"
- board text added: "External ports"
- board text added: "I2C ports"
- board text added: "SMART HOME v1.1"
- board text added: "Sensor board"

Commit message: Creating charts
Parts:
- C1, C6: value (none) -> 100u
- C14, C15, C2, C3, C4, C5, C7: value (none) -> 10u
- R10: value (none) -> 330
- R17, R20: value (none) -> 20K
- R18, R19: value (none) -> 10K
- R30: value (none) -> 100

Commit message: Add new method of controling the supply
Parts:
- removed C7: 10u, rcl:C0805K
- removed R21, R22, R23, R24: (no value), rcl:R0805
- removed U2: LM3940IMP-3.3, LM3940IMP-3.3:SOT230P700X180-4N
- added OK1: 4N35, optocoupler:DIL06
- added R34, R35, R36: (no value), rcl:R0805
- C6: value 100u -> (none)
- moved C6 114.5 mm to (-19.4, -25.1), flipped to the top
Connections:
- removed net N$15: J4.2, R23.1
- removed net N$21: J3.2, R21.1
- new net EN_5V: R35.2
- new net N$25: IC2.5, OK1.5, R34.1
- new net N$26: OK1.1, R35.1
- new net N$28: U1.13
- new net N$29: C6.2, OK1.6, R36.2
- net +3V3: no longer C7.1, U2.3
- net +5V: no longer C6.1, U2.1
- net A2: now also J3.2; no longer R21.2, R22.1
- net A3: now also J4.2; no longer R23.2, R24.1
- net GND: now also C6.1, OK1.2, OK1.4, R36.1; no longer C6.2, C7.2, IC2.5, R22.2, R24.2, U2.2, U2.4
- net VCC: now also R34.2
Routing:
- net GND: track 77.2 -> 69.9 mm
- net N$15: track 6.08 -> 0.00 mm
- net N$21: track 5.29 -> 0.00 mm
- net A3: track 48.3 -> 44.8 mm
- net +3V3: track 248.8 -> 246.0 mm
- net +5V: track 246.4 -> 243.9 mm
- net A2: track 39.6 -> 39.0 mm

Commit message: Finished PCB Sensor
Parts:
- added C16: 10u, rcl:E3,5-8
- added C17: 22u, rcl:C0805K
- added C18: 100p, rcl:C0805K
- added C7: 100u, rcl:E2,5-6
- added D1: 1N5822, diode:C4111-15
- added IC1: LM2576S, v-reg-3:TO263-5
- added L2: DE1207-100, ferrocore:DE1207
- added R21, R22: (no value), rcl:R0805
- moved R35 86.8 mm to (30.5, 53.6), turned to 180 degrees
- moved C6 86.7 mm to (22.0, 51.1)
- moved R36 85.3 mm to (21.9, 53.1)
- moved R34 80.7 mm to (17.4, 58.5), turned to 90 degrees
- moved OK1 74.2 mm to (24.8, 58.2), turned to 90 degrees
- moved I2C_3V3_2 27.8 mm to (26.2, 7.16)
- moved R26 22.8 mm to (35.4, 17.2)
- moved J7 20.2 mm to (65.9, 41.4)
- moved C12 19.3 mm to (38.2, 16.2), turned to 180 degrees
- moved R3 18.3 mm to (62.0, 39.5)
- moved J6 18.2 mm to (66.0, 33.4)
- moved Q3 18.2 mm to (59.4, 41.5)
- moved C3 17.9 mm to (62.0, 43.7)
- moved R11 17.9 mm to (56.8, 43.8)
- moved R12 17.6 mm to (56.8, 39.6)
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Connections:
- removed net N$28: U1.13
- new net N$21: D1.C, IC1.2, L2.1
- new net N$30: IC1.4, R21.2, R22.1
- net +3V3: now also C16.+, C17.2, C18.2, L2.2, R22.2
- net EN_5V: now also U1.13
- net GND: now also C16.-, C17.1, C18.1, C7.-, D1.A, IC1.3, IC1.5, R21.1
- net VCC: now also C7.+, IC1.1
Routing:
- net VCC: track 24.3 -> 96.9 mm
- net GND: track 69.9 -> 26.3 mm, vias 6 -> 55
- net EN_5V: track 0.00 -> 34.6 mm, vias 0 -> 2
- net +5V: track 243.9 -> 278.2 mm, vias 4 -> 3
- net +3V3: track 246.0 -> 275.6 mm
- net SDA_LV: track 91.4 -> 63.6 mm, vias 1 -> 3
- net N$21: track 0.00 -> 27.8 mm, vias 0 -> 1
- net A3: track 44.8 -> 23.0 mm, vias 0 -> 2
- net SCL_LV: track 92.9 -> 71.7 mm, vias 1 -> 2
- net N$25: track 0.00 -> 20.8 mm
- net SCL: track 35.6 -> 15.5 mm
- net A2: track 39.0 -> 25.3 mm
- net SDA: track 25.3 -> 14.9 mm
- net K4: track 14.3 -> 21.7 mm
- net N$19: track 42.1 -> 34.9 mm
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Other:
- board size 75 x 71.2 mm -> 73.3 x 77 mm
- board text added: "Arkadiusz"
- board text added: "Kruszyński"
- board text added: "SMART HOME v1.2"
- board text removed: "A. KRUSZYNSKI"
- board text removed: "C.KULCZYK"
- board text removed: "SMART HOME v1.1"
