File: PCB/ESPSensor/Płytka.sch (EAGLE design)
At the start: 84 parts, among them IC2 LM2576S/5V, J1 HUM1, J2 HUM2, J3 TEMP, J4 SUN, J5 K3, J6 K2, J7 K1, J8 K5, J9 K4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

Commit message: Add new method of controling the supply
Parts:
- removed C7: 10u, rcl:C-EUC0805K
- removed R21, R22, R23, R24: (no value), rcl:R-EU_R0805
- removed U2: LM3940IMP-3.3, LM3940IMP-3.3:LM3940IMP-3.3
- added OK1: 4N35, optocoupler:4N35
- added R34, R35, R36: (no value), rcl:R-EU_R0805
- C6: value 100u -> (none)
Connections:
- removed net N$15: J4.2, R23.1
- removed net N$21: J3.2, R21.1
- new net EN_5V: R35.2
- new net N$25: IC2.OFF, OK1.COL, R34.1
- new net N$26: OK1.A, R35.1
- new net N$28: U1.IO14
- new net N$29: C6.2, OK1.BAS, R36.2
- net +3V3: no longer C7.1, U2.OUT
- net +5V: no longer C6.1, U2.IN
- net A2: now also J3.2; no longer R21.2, R22.1
- net A3: now also J4.2; no longer R23.2, R24.1
- net GND: now also C6.1, OK1.C, OK1.EMI, R36.1; no longer C6.2, C7.2, IC2.OFF, R22.2, R24.2, U2.GND
- net VCC: now also R34.2
Other:
- moved on the sheet: C10, C11, C6, C9, D5, D6, D7, J2, J3, R18, R19, R20

Commit message: Finished PCB Sensor
Parts:
- added C16: 10u, rcl:CPOL-EUE3.5-8
- added C17: 22u, rcl:C-EUC0805K
- added C18: 100p, rcl:C-EUC0805K
- added C7: 100u, rcl:CPOL-EUE2.5-6
- added D1: 1N5822, diode:1N5908
- added IC1: LM2576S, v-reg-3:LM2576S
- added L2: DE1207-100, ferrocore:DE1207-100
- added R21, R22: (no value), rcl:R-EU_R0805
Connections:
- removed net N$28: U1.IO14
- new net N$21: D1.C, IC1.OUT, L2.1
- new net N$30: IC1.FB, R21.2, R22.1
- net +3V3: now also C16.+, C17.2, C18.2, L2.2, R22.2
- net EN_5V: now also U1.IO14
- net GND: now also C16.-, C17.1, C18.1, C7.-, D1.A, IC1.GND, IC1.OFF, R21.1
- net VCC: now also C7.+, IC1.VIN
Other:
- moved on the sheet: C6, LED1, LED5, OK1, R10, R30, R35, R36, SUPPLY-1, SUPPLY-2, SV2
